Commit message: fix(tf): add URDF sensor frames and replace static_transform_publishers with robot_state_publisher

File: src/Tyre_Inspection_Bot/src/amr_hardware/src/ugv_description/urdf/ugv_rover.urdf (robot description, URDF)
Before this commit: robot ugv_rover, 13 links, 12 joints
Links:
- added link camera_depth_optical_frame, mass 0.001
- added link camera_left, mass 0.05
- added link camera_right, mass 0.05
- added link imu_link, mass 0.01
Joints:
- added joint camera_depth_optical_joint: type fixed, parent camera_left, child camera_depth_optical_frame, origin xyz=0 0 0 rpy=0 0 0
- added joint camera_left_joint: type fixed, parent base_link, child camera_left, origin xyz=0.0418 0.03 0 rpy=-1.5708 0 -1.5708
- added joint camera_right_joint: type fixed, parent camera_left, child camera_right, origin xyz=0.06 0 0 rpy=0 0 0
- added joint imu_joint_aurora: type fixed, parent camera_left, child imu_link, origin xyz=0.03 0 0 rpy=0 0 -1.5708
